Commit message: second stella git

File: stella_description/urdf/macros.xacro (robot description, xacro)
@@ -19,5 +19,5 @@
 	/>
 </macro>
-<macro name="wheel" params="lr tY stl_file">
+<macro name="wheel" params="lr tY">
 <link name="${lr}_wheel">
   <collision>
@@ -30,5 +30,5 @@
     <origin xyz="0 0 0" rpy="0 ${PI/2} ${PI/2}" />
     <geometry>
-    <mesh filename="${stl_file}" scale="0.001 0.001 0.001"/>
+      <cylinder length="${wheelWidth}" radius="${wheelRadius}"/>
     </geometry>
     <material name="black"/>

File: stella_description/urdf/stella.xacro (robot description, xacro)
@@ -25,6 +25,7 @@
 			<origin xyz="0 0 ${wheelRadius}" rpy="0 0 0"/>
 			<geometry>
-				<mesh filename="package://stella_description/meshes/bases/stella_base.stl" scale="0.001 0.001 0.001"/>
+				<box size="${bodyLength} ${bodyWidth} ${bodyHeight}"/>
 			</geometry>
+			<material name="grey"/>
 		</visual>
 		<collision>
@@ -56,5 +57,5 @@
     <origin xyz="${-wheelRadius - 0.02 + bodyLength/2} 0 ${-bodyHeight / 2 + bodyToFloorHeight +  wheelRadius}" rpy="0 0 0"/>
     <geometry>
-      <mesh filename="package://stella_description/meshes/wheels/caster_wheel.stl" scale="0.001 0.001 0.001"/>
+      <sphere radius="${wheelRadius}"/>
     </geometry>
     <material name="black"/>
@@ -66,6 +67,6 @@
   </inertial>
 </link>
-<wheel lr="left" tY="1" stl_file="package://stella_description/meshes/wheels/left_wheel.stl"/>
-<wheel lr="right" tY="-1" stl_file="package://stella_description/meshes/wheels/right_wheel.stl"/>
+<wheel lr="left" tY="1"/>
+<wheel lr="right" tY="-1"/>
  <joint name="imu_joint" type="fixed">
     <parent link="base_link"/>
@@ -83,5 +84,5 @@
       <origin xyz="0 0 0.0" rpy="0 0 0"/>
       <geometry>
-        <mesh filename="package://stella_description/meshes/sensors/rplidar.stl" scale="0.001 0.001 0.001"/>
+        <mesh filename="package://stella_description/meshes/sensors/lds.stl" scale="0.001 0.001 0.001"/>
       </geometry>
       <material name="dark"/>
